Commit message: update

File: autosim/urdf/husky.urdf (robot description, URDF)
Before this commit: robot husky, 9 links, 8 joints
Links:
- added link camera_link, mass 0.2; collision box size=0.05 0.05 0.04; visual box size=0.05 0.05 0.04
Joints:
- added joint camera_joint: type fixed, parent base_link, child camera_link, origin xyz=0.20 0 0.32 rpy=0 0 0

File: autosim/urdf/turtlebot3_burger.urdf (robot description, URDF)
Before this commit: robot turtlebot3_burger, 8 links, 7 joints
Links:
- added link camera_link, mass 0.08; collision box size=0.04 0.04 0.03; visual box size=0.04 0.04 0.03
Joints:
- added joint camera_joint: type fixed, parent base_link, child camera_link, origin xyz=0.03 0 0.20 rpy=0 0 0
