Commit message: [feat] update

File: automanip/examples/quadrotor/urdf/quadrotor.urdf (robot description, URDF)
Before this commit: robot quadrotor, 11 links, 10 joints
Links:
- removed link body
- removed link dx
- removed link dy
- removed link dz
- removed link pitch_link
- removed link rotor_fl
- removed link rotor_fr
- removed link rotor_rl
- removed link rotor_rr
- removed link world
- removed link yaw_link
- added link base, mass 0.5; visual mesh filename=package://ocs2_robotic_assets/resources/quadrotor/meshes/qu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 scale=0.4 0.4 0.4
Joints:
- removed joint arm_fl
- removed joint arm_fr
- removed joint arm_rl
- removed joint arm_rr
- removed joint pitch
- removed joint roll
- removed joint x
- removed joint y
- removed joint yaw
- removed joint z
