Commit message: [feat] update

File: autosim/robot/husky/husky.urdf (robot description, URDF)
Before this commit: robot husky, 10 links, 9 joints
Links:
- link base_link: mass 50.0 -> 46.034; geometry collision box size=0.987 0.570 0.220; visual mesh filename=meshes/base_link.dae
- link front_left_wheel_link: mass 2.5 -> 2.637; geometry collision cylinder length=0.1143 radius=0.1651; visual mesh filename=meshes/wheel.dae
- link front_right_wheel_link: mass 2.5 -> 2.637; geometry collision cylinder length=0.1143 radius=0.1651; visual mesh filename=meshes/wheel.dae
- link imu_link: geometry 
- link rear_left_wheel_link: mass 2.5 -> 2.637; geometry collision cylinder length=0.1143 radius=0.1651; visual mesh filename=meshes/wheel.dae
- link rear_right_wheel_link: mass 2.5 -> 2.637; geometry collision cylinder length=0.1143 radius=0.1651; visual mesh filename=meshes/wheel.dae
Joints:
- joint base_joint: origin xyz=0 0 0.165 rpy=0 0 0 -> xyz=0 0 0.1651 rpy=0 0 0
- joint front_left_wheel_joint: axis 0 0 1 -> 0 1 0; origin xyz=0.256 0.285 -0.0 rpy=-1.57079632679 0 0 -> xyz=0.256 0.285 0 rpy=0 0 0
- joint front_right_wheel_joint: axis 0 0 1 -> 0 1 0; origin xyz=0.256 -0.285 -0.0 rpy=-1.57079632679 0 0 -> xyz=0.256 -0.285 0 rpy=0 0 0
- joint rear_left_wheel_joint: axis 0 0 1 -> 0 1 0; origin xyz=-0.256 0.285 -0.0 rpy=-1.57079632679 0 0 -> xyz=-0.256 0.285 0 rpy=0 0 0
- joint rear_right_wheel_joint: axis 0 0 1 -> 0 1 0; origin xyz=-0.256 -0.285 -0.0 rpy=-1.57079632679 0 0 -> xyz=-0.256 -0.285 0 rpy=0 0 0

File: autosim/robot/turtlebot3_burger/turtlebot3_burger.urdf (robot description, URDF)
Before this commit: robot turtlebot3_burger, 9 links, 8 joints
Links:
- link base_link: mass 1.0 -> 0.82573504; geometry collision box size=0.140 0.140 0.143; visual mesh filename=meshes/bases/burger_base.stl scale=0.001 0.001 0.001
- link base_scan: geometry collision cylinder length=0.0315 radius=0.055; visual mesh filename=meshes/sensors/lds.stl scale=0.001 0.001 0.001
- link caster_back_link: geometry collision box size=0.030 0.009 0.020
- link imu_link: geometry 
- link wheel_left_link: mass 0.028 -> 0.02849894; geometry collision cylinder length=0.018 radius=0.033; visual mesh filename=meshes/wheels/left_tire.stl scale=0.001 0.001 0.001
- link wheel_right_link: mass 0.028 -> 0.02849894; geometry collision cylinder length=0.018 radius=0.033; visual mesh filename=meshes/wheels/right_tire.stl scale=0.001 0.001 0.001
Joints:
- joint caster_back_joint: origin xyz=-0.081 0 -0.004 rpy=0 0 0 -> xyz=-0.081 0 -0.004 rpy=-1.57079632679 0 0
- joint imu_joint: origin xyz=0 0 0.068 rpy=0 0 0 -> xyz=-0.032 0 0.068 rpy=0 0 0
- joint scan_joint: origin xyz=-0.032 0 0.5 rpy=0 0 0 -> xyz=-0.032 0 0.172 rpy=0 0 0

File: autosim/robot/turtlebot3_burger/turtlebot3_burger_bev.urdf (robot description, URDF)
Before this commit: robot turtlebot3_burger_bev, 15 links, 14 joints
Links:
- link base_link: mass 1.0 -> 0.82573504; geometry collision box size=0.140 0.140 0.143; visual mesh filename=meshes/bases/burger_base.stl scale=0.001 0.001 0.001
- link base_scan: geometry collision cylinder length=0.0315 radius=0.055; visual mesh filename=meshes/sensors/lds.stl scale=0.001 0.001 0.001
- link caster_back_link: geometry collision box size=0.030 0.009 0.020
- link imu_link: geometry 
- link wheel_left_link: mass 0.028 -> 0.02849894; geometry collision cylinder length=0.018 radius=0.033; visual mesh filename=meshes/wheels/left_tire.stl scale=0.001 0.001 0.001
- link wheel_right_link: mass 0.028 -> 0.02849894; geometry collision cylinder length=0.018 radius=0.033; visual mesh filename=meshes/wheels/right_tire.stl scale=0.001 0.001 0.001
Joints:
- joint caster_back_joint: origin xyz=-0.081 0 -0.004 rpy=0 0 0 -> xyz=-0.081 0 -0.004 rpy=-1.57079632679 0 0
- joint imu_joint: origin xyz=0 0 0.068 rpy=0 0 0 -> xyz=-0.032 0 0.068 rpy=0 0 0
- joint scan_joint: origin xyz=-0.032 0 0.5 rpy=0 0 0 -> xyz=-0.032 0 0.172 rpy=0 0 0
